File: Embedded.X/scheme/project/project.sch (KiCad schematic (older format))
At the start: 8 parts, among them SW1 Pause, SW2 Rotate, SW3 Left, SW4 Right, SW5 Down, U1 PIC16F884

Commit message: Added a PCB and fixed up the scheme
Parts:
- removed DS1: LCD, Display:AG12864E, symbol mylib:LCD
- removed RV1: 10k, symbol Device:R_POT_TRIM
- removed SW1: Pause, symbol Switch:SW_MEC_5G
- removed SW2: Rotate, symbol Switch:SW_MEC_5G
- removed SW3: Left, symbol Switch:SW_MEC_5G
- removed SW4: Right, symbol Switch:SW_MEC_5G
- removed SW5: Down, symbol Switch:SW_MEC_5G
- added SW1: Pause, Button_Switch_THT:SW_PUSH_6mm, symbol Switch:SW_SPST
- added SW2: Rotate, Button_Switch_THT:SW_PUSH_6mm, symbol Switch:SW_SPST
- added SW3: Right, Button_Switch_THT:SW_PUSH_6mm, symbol Switch:SW_SPST
- added SW4: Left, Button_Switch_THT:SW_PUSH_6mm, symbol Switch:SW_SPST
- added SW5: Down, Button_Switch_THT:SW_PUSH_6mm, symbol Switch:SW_SPST
- added SW6: Power_sw, Button_Switch_THT:SW_Slide_1P2T_CK_OS102011MS2Q, symbol mylib:SW_SPDT
- U1: footprint (none) -> Package_DIP:DIP-40_W15.24mm; symbol mylib:PIC -> project-rescue:PIC-mylib
Connections:
- net GND: now also SW1.2 (B), SW2.2 (B), SW3.2 (B), SW4.2 (B), SW5.2 (B), SW6.3 (C)
- net VCC: now also SW6.1 (A); no longer U1.11 (VDD)
- net nCS1: now reaches U1.16 (T1OSI/CCP2/RC1)
- net DB1: now reaches U1.3 (C12IN1-/AN1/RA1)
- net DB2: now reaches U1.4 (C2IN+/CVref/Vref-/AN2/RA2)
- net DB3: now reaches U1.5 (C1IN+/Vref+/AN3/RA3)
- net DB4: now reaches U1.6 (C1OUT/T0CKI/RA4)
- net DB5: now reaches U1.7 (C2OUT/~SS~/AN4/RA5)
- net DB6: now reaches U1.14 (RA6/OSC2/CLKOUT)
- net DB7: now reaches U1.13 (RA7/OSC1/CLKIN)
- net nRST: now reaches U1.20 (RD1)
- net nCS2: now reaches U1.15 (T10S0/T1CKI/RC0)
- net DnI: now reaches U1.17 (P1A/CCP1/RC2)
- net RnW: now reaches U1.18 (SCL/SCK/RC3)
- net E: now reaches U1.19 (RD0)
- net DB0: now reaches U1.2 (C12IN0-/ULPWU/AN0/RA0)
- net at U1.33 (INT/AN12/RB0): now also SW1.1 (A)
- net at U1.34 (C12IN3-/AN10/RB1): now also SW2.1 (A)
- net at U1.35 (AN8/RB2): now also SW3.1 (A)
- net at U1.36 (C12IN2-/PGM/AN9/RB3): now also SW4.1 (A)
- net at U1.37 (AN11/RB4): now also SW5.1 (A)
- net at U1.1 (RE3/~MCLR~/Vpp): now also U1.11 (VDD), SW6.2 (B)
- no-connect marks 21 -> 32
